Commit message: changes

File: description/depth_camera.xacro (robot description, xacro)
@@ -13,9 +13,4 @@
             <material name="red"/>
         </visual>
-        <collision>
-            <geometry>
-                <box size="0.02 0.08 0.08"/>
-            </geometry>
-        </collision>
     </link>
     <joint name="camera_optical_joint" type="fixed">
@@ -35,6 +30,6 @@
                 <image>
                     <format>B8G8R8</format>
-                    <width>840</width>
-                    <height>680</height>
+                    <width>640</width>
+                    <height>480</height>
                 </image>
                 <clip>
@@ -46,5 +41,5 @@
                 <frame_name>camera_link_optical</frame_name>
                 <min_depth>0.1</min_depth>
-                <max_depth>100</max_depth>
+                <max_depth>100.0</max_depth>
             </plugin>
         </sensor>

File: description/lidar.xacro (robot description, xacro)
@@ -9,5 +9,5 @@
         <visual>
             <geometry>
-              <cylinder radius="0.06" length="0.06"/>
+              <cylinder radius="0.05" length="0.06"/>
             </geometry>
             <material name="red"/>
@@ -15,8 +15,8 @@
           <collision>
             <geometry>
-              <cylinder radius="0.06" length="0.06"/>
+              <cylinder radius="0.05" length="0.06"/>
             </geometry>
           </collision>
-          <xacro:inertial_cylinder mass="1" length="0.06" radius="0.06">
+          <xacro:inertial_cylinder mass="1" length="0.06" radius="0.05">
             <origin xyz="0 0 0" rpy="0 0 0"/>
           </xacro:inertial_cylinder>

File: description/robot.urdf.xacro (robot description, xacro)
@@ -2,7 +2,7 @@
 <robot xmlns:xacro="http://www.ros.org/wiki/xacro"  name="robot">
     <xacro:include filename="robot_core.xacro" />
-    <xacro:include filename="gazebo_control.xacro" />
-    <!-- <xacro:include filename="ros2_control.xacro" /> -->
-    <xacro:include filename="lidar.xacro" />
+    <!-- <xacro:include filename="gazebo_control.xacro" /> -->
+    <xacro:include filename="ros2_control.xacro" />
+    <!-- <xacro:include filename="lidar.xacro" /> -->
     <xacro:include filename="camera.xacro" />
     <!-- <xacro:include filename="depth_camera.xacro" /> -->
