Commit message: vaerious changes

File: description/camera.xacro (robot description, xacro)
@@ -19,4 +19,5 @@
         </collision>
     </link>
+<div id="TODO"> camera link</div>
     <joint name="camera_optical_joint" type="fixed">
         <parent link="camera_link"/>

File: description/robot.urdf.xacro (robot description, xacro)
@@ -1,8 +1,13 @@
 <?xml version="1.0"?>
 <robot xmlns:xacro="http://www.ros.org/wiki/xacro"  name="robot">
+    <xacro:arg name="use_ros2_control" default="true"/>
     <xacro:include filename="robot_core.xacro" />
-    <!-- <xacro:include filename="gazebo_control.xacro" /> -->
-    <xacro:include filename="ros2_control.xacro" />
-    <!-- <xacro:include filename="lidar.xacro" /> -->
+    <xacro:if value="$(arg use_ros2_control)">
+        <xacro:include filename="ros2_control.xacro" />
+    </xacro:if>
+    <xacro:unless value="$(arg use_ros2_control)">
+        <xacro:include filename="gazebo_control.xacro" />
+    </xacro:unless>
+    <xacro:include filename="lidar.xacro" />
     <xacro:include filename="camera.xacro" />
     <!-- <xacro:include filename="depth_camera.xacro" /> -->

File: description/robot_core.xacro (robot description, xacro)
@@ -70,5 +70,5 @@
     <collision>
       <geometry>
-        <cylinder radius="${wheel_radius}" length="${wheel_length}"/>
+        <sphere radius="${wheel_radius}"/>
       </geometry>
     </collision>
@@ -98,5 +98,5 @@
     <collision>
       <geometry>
-        <cylinder radius="${wheel_radius}" length="${wheel_length}"/>
+        <sphere radius="${wheel_radius}"/>
       </geometry>
     </collision>
@@ -126,5 +126,5 @@
     <collision>
       <geometry>
-        <cylinder radius="${wheel_radius}" length="${wheel_length}"/>
+        <sphere radius="${wheel_radius}"/>
       </geometry>
     </collision>
@@ -154,5 +154,5 @@
     <collision>
       <geometry>
-        <cylinder radius="${wheel_radius}" length="${wheel_length}"/>
+        <sphere radius="${wheel_radius}"/>
       </geometry>
     </collision>
